Commit message: 跑通cas02

File: resources/CAS02/urdf/CB02_URDF(ECS-WK)-1.urdf (robot description, URDF)
Before this commit: robot CB02_URDF(ECS-WK)-1, 28 links, 27 joints
Links:
- link base_link: geometry visual mesh filename=../meshes/base_link.STL
- link left_leg_ankle_pitch_link: geometry visual mesh filename=../meshes/left_leg_ankle_pitch_link.STL
- link left_leg_ankle_roll_link: geometry collision box size=0.23 0.08 0.02; visual mesh filename=../meshes/left_leg_ankle_roll_link.STL
- link left_leg_knee_pitch_link: geometry collision box size=0.03 0.06 0.1; collision box size=0.05 0.07 0.19
- link left_leg_pelvic_pitch_link: geometry visual mesh filename=../meshes/left_leg_pelvic_pitch_link.STL
- link left_shoulder_pitch_link: geometry visual mesh filename=../meshes/left_shoulder_pitch_link.STL
- link right_leg_ankle_pitch_link: geometry visual mesh filename=../meshes/right_leg_ankle_pitch_link.STL
- link right_leg_ankle_roll_link: geometry collision box size=0.23 0.08 0.02; visual mesh filename=../meshes/right_leg_ankle_roll_link.STL
- link right_leg_knee_pitch_link: geometry collision box size=0.03 0.06 0.1; collision box size=0.05 0.07 0.19
- link right_leg_pelvic_pitch_link: geometry visual mesh filename=../meshes/right_leg_pelvic_pitch_link.STL
- link right_shoulder_pitch_link: geometry visual mesh filename=../meshes/right_shoulder_pitch_link.STL
- link waist_yaw_link: geometry collision box size=0.15 0.2 0.3; visual mesh filename=../meshes/waist_yaw_link.STL
Joints:
- joint head_pitch_joint: type revolute -> fixed
- joint left_shoulder_roll_joint: origin xyz=0 0.057 0 rpy=0 0 0 -> xyz=0 0.057 0 rpy=0.1745 0 0
- joint left_wrist_yaw_joint: type revolute -> fixed
- joint right_shoulder_roll_joint: origin xyz=0 -0.057 0 rpy=0 0 0 -> xyz=0 -0.057 0 rpy=-0.1745 0 0
- joint right_wrist_yaw_joint: type revolute -> fixed

Commit message: gaiurdf

File: resources/CAS02/urdf/CB02_URDF(ECS-WK)-1.urdf (robot description, URDF)
Before this commit: robot CB02_URDF(ECS-WK)-1, 28 links, 27 joints
Links:
- link head_pitch_link: geometry collision sphere radius=0.07; visual mesh filename=../meshes/head_pitch_link.STL
- link head_yaw_link: geometry visual mesh filename=../meshes/head_yaw_link.STL
- link left_leg_knee_pitch_link: geometry collision box size=0.03 0.06 0.1; collision box size=0.05 0.07 0.19
- link left_leg_pelvic_pitch_link: geometry collision cylinder length=0.08 radius=0.06; visual mesh filename=../meshes/left_leg_pelvic_pitch_link.STL
- link left_leg_pelvic_roll_link: geometry visual mesh filename=../meshes/left_leg_pelvic_roll_link.STL
- link left_leg_pelvic_yaw_link: geometry visual mesh filename=../meshes/left_leg_pelvic_yaw_link.STL
- link right_leg_knee_pitch_link: geometry collision box size=0.03 0.06 0.1; collision box size=0.05 0.07 0.19
- link right_leg_pelvic_pitch_link: geometry collision cylinder length=0.08 radius=0.06; visual mesh filename=../meshes/right_leg_pelvic_pitch_link.STL
- link right_leg_pelvic_roll_link: geometry visual mesh filename=../meshes/right_leg_pelvic_roll_link.STL
- link right_leg_pelvic_yaw_link: geometry visual mesh filename=../meshes/right_leg_pelvic_yaw_link.STL
